File: pie-shield.brd (EAGLE design)
At the start: 35.5 x 56.2 mm, 15 parts, among them IC6 78L05, IC8 MAX487, X6 RJ45-8L-B

Commit message: using uart pins
Connections:
- net GND: now also U$2.P1_9
- net RXD_AL: now also U$2.P1_10; no longer U$2.P5_5
- net SELECT: now also U$2.P1_11; no longer U$2.P5_6
- net TXD_AL: now also U$2.P1_8; no longer U$2.P5_4
Routing:
- net TXD_AL: track 12.7 -> 20.4 mm
- net SELECT: track 14.8 -> 18.9 mm
- net RXD_AL: track 26.3 -> 29.5 mm
Changed lines of the file:
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@@
 <signal name="RXD_AL">
 <contactref element="OK2" pad="6"/>
-<contactref element="U$2" pad="P5_5"/>
-<wire x1="12.7" y1="48.26" x2="13.97" y2="46.99" width="0.4064" layer="1"/>
-<wire x1="13.97" y1="46.99" x2="22.86" y2="46.99" width="0.4064" layer="1"/>
 <wire x1="22.86" y1="46.99" x2="31.115" y2="38.735" width="0.4064" layer="1"/>
 <wire x1="31.115" y1="38.735" x2="31.115" y2="34.8234" width="0.4064" layer="1"/>
+<contactref element="U$2" pad="P1_10"/>
+<wire x1="12.7" y1="53.34" x2="13.97" y2="52.07" width="0.4064" layer="1"/>
+<wire x1="13.97" y1="52.07" x2="18.415" y2="52.07" width="0.4064" layer="1"/>
+<wire x1="18.415" y1="52.07" x2="19.05" y2="51.435" width="0.4064" layer="1"/>
+<wire x1="19.05" y1="51.435" x2="19.05" y2="49.53" width="0.4064" layer="1"/>
+<wire x1="22.86" y1="46.99" x2="21.59" y2="46.99" width="0.4064" layer="1"/>
+<wire x1="21.59" y1="46.99" x2="19.05" y2="49.53" width="0.4064" layer="1"/>
 </signal>
 <signal name="TXD_AL">
 <contactref element="OK1" pad="3"/>
-<contactref element="U$2" pad="P5_4"/>
-<wire x1="10.16" y1="45.72" x2="14.605" y2="41.275" width="0.4064" layer="1"/>
 <wire x1="14.605" y1="41.275" x2="14.605" y2="34.8234" width="0.4064" layer="1"/>
+<contactref element="U$2" pad="P1_8"/>
+<wire x1="10.16" y1="53.34" x2="11.43" y2="52.07" width="0.4064" layer="1"/>
+<wire x1="11.43" y1="52.07" x2="11.43" y2="44.45" width="0.4064" layer="1"/>
+<wire x1="11.43" y1="44.45" x2="14.605" y2="41.275" width="0.4064" layer="1"/>
 </signal>
 <signal name="N$37">
@@
 <signal name="SELECT">
 <contactref element="OK3" pad="3"/>
-<contactref element="U$2" pad="P5_6"/>
-<wire x1="12.7" y1="45.72" x2="22.225" y2="36.195" width="0.4064" layer="1"/>
-<wire x1="22.225" y1="36.195" x2="22.225" y2="34.8234" width="0.4064" layer="1"/>
+<wire x1="22.225" y1="36.195" x2="22.225" y2="35.56" width="0.4064" layer="1"/>
+<contactref element="U$2" pad="P1_11"/>
+<wire x1="22.225" y1="35.56" x2="22.225" y2="34.8234" width="0.4064" layer="1"/>
+<wire x1="15.24" y1="50.8" x2="22.225" y2="43.815" width="0.4064" layer="1"/>
+<wire x1="22.225" y1="43.815" x2="22.225" y2="36.195" width="0.4064" layer="1"/>
 </signal>
 <signal name="GND">
@@
 <contactref element="U$2" pad="P5_7"/>
 <contactref element="U$2" pad="P1_6"/>
+<contactref element="U$2" pad="P1_9"/>
 </signal>
 </signals>
